Commit message: Update camera.xacro

File: urdf2/final_description/urdf/camera.xacro (robot description, xacro)
@@ -1,33 +1,90 @@
 <?xml version="1.0"?>
-<robot xmlns:xacro="http://www.ros.org/wiki/xacro">
-    <link name="camera_link"></link>
+<robot xmlns:xacro="http://www.ros.org/wiki/xacro" >
+    <joint name="camera_joint" type="fixed">
+        <parent link="runner_plate_v1_1"/>
+        <child link="camera_link"/>
+        <origin xyz="0.276 0 0.181" rpy="0 0.18 0"/>
+    </joint>
+    <link name="camera_link">
+        <visual>
+            <geometry>
+                <box size="0.010 0.03 0.03"/>
+            </geometry>
+            <material name="black"/>
+        </visual>
+        <visual>
+            <origin xyz="0 0 -0.05"/>
+            <geometry>
+                <cylinder radius="0.002" length="0.1"/>
+            </geometry>
+            <material name="black"/>
+        </visual>
+    </link>
+    <joint name="camera_optical_joint" type="fixed">
+        <parent link="camera_link"/>
+        <child link="camera_link_optical"/>
+        <origin xyz="0 0 0" rpy="${-pi/2} 0 ${-pi/2}"/>
+    </joint>
     <link name="camera_link_optical"></link>
-    <joint name="camera_joint" type="fixed">
-        <origin xyz="0.05 0.22 0" rpy="${-pi/2} ${pi} ${-pi/2}" />
-        <parent link="base_link" />
-        <child link="camera_link" />
+    <gazebo reference="camera_link">
+        <material>white</material>
+        <sensor name="camera" type="camera">
+            <pose> 0 0 0 1.57 0 0 </pose>
+            <visualize>true</visualize>
+            <update_rate>10</update_rate>
+            <camera>
+                <horizontal_fov>1.089</horizontal_fov>
+                <image>
+                    <format>R8G8B8</format>
+                    <width>640</width>
+                    <height>480</height>
+                </image>
+                <clip>
+                    <near>0.05</near>
+                    <far>8.0</far>
+                </clip>
+                <ignition_frame_id>camera_link_optical</ignition_frame_id>
+            </camera>
+        </sensor>
+    </gazebo>
+    <joint name="depth_camera_joint" type="fixed">
+        <parent link="runner_plate_v1_2"/>
+        <child link="depth_camera_link"/>
+        <origin xyz="0.305 0 0.08" rpy="0 0 0"/>
     </joint>
-    <joint name="camera_optical_joint" type="fixed">
-        <origin xyz="0 0 0" rpy="${-pi/2} 0 ${-pi/2}" />
-        <parent link="camera_link" />
-        <child link="camera_link_optical" />
+    <link name="depth_camera_link">
+        <visual>
+            <geometry>
+                <box size="0.010 0.03 0.03"/>
+            </geometry>
+            <material name="orange"/>
+        </visual>
+    </link>
+    <joint name="depth_camera_optical_joint" type="fixed">
+        <parent link="depth_camera_link"/>
+        <child link="depth_camera_link_optical"/>
+        <origin xyz="0 0 0" rpy="${-pi/2} 0 ${-pi/2}"/>
     </joint>
-    <gazebo reference="camera_link">
+    <link name="depth_camera_link_optical"></link>
+    <gazebo reference="depth_camera_link">
+        <material>orange</material>
         <sensor name="depth_camera" type="depth">
-            <topic>depth</topic>
             <pose> 0 0 0 0 0 0 </pose>
             <visualize>true</visualize>
-            <always_on>1</always_on>
             <update_rate>10</update_rate>
             <camera>
-                <horizontal_fov>1.134</horizontal_fov>
+                <horizontal_fov>1.089</horizontal_fov>
                 <image>
-                    <width>800</width>
-                    <height>600</height>
+                    <format>B8G8R8</format>
+                    <width>640</width>
+                    <height>480</height>
                 </image>
                 <clip>
-                    <near>0.45</near>
-                    <far>3.0</far>
+                    <near>0.05</near>
+                    <far>8.0</far>
                 </clip>
+                <ignition_frame_id>depth_camera_link_optical</ignition_frame_id>
+                <min_depth>0.1</min_depth>
+                <max_depth>100.0</max_depth>
             </camera>
         </sensor>

Commit message: added sensors

File: urdf2/final_description/urdf/camera.xacro (robot description, xacro)
@@ -4,5 +4,5 @@
         <parent link="runner_plate_v1_1"/>
         <child link="camera_link"/>
-        <origin xyz="0.276 0 0.181" rpy="0 0.18 0"/>
+        <origin xyz="-0.05 0 0.075" rpy="0 -1.57 0"/>
     </joint>
     <link name="camera_link">
@@ -11,12 +11,5 @@
                 <box size="0.010 0.03 0.03"/>
             </geometry>
-            <material name="black"/>
-        </visual>
-        <visual>
-            <origin xyz="0 0 -0.05"/>
-            <geometry>
-                <cylinder radius="0.002" length="0.1"/>
-            </geometry>
-            <material name="black"/>
+            <material name="blue"/>
         </visual>
     </link>
@@ -24,5 +17,5 @@
         <parent link="camera_link"/>
         <child link="camera_link_optical"/>
-        <origin xyz="0 0 0" rpy="${-pi/2} 0 ${-pi/2}"/>
+        <origin xyz="0 0 0" rpy="0 0 0"/>
     </joint>
     <link name="camera_link_optical"></link>
@@ -49,7 +42,7 @@
     </gazebo>
     <joint name="depth_camera_joint" type="fixed">
-        <parent link="runner_plate_v1_2"/>
+        <parent link="runner_plate_v1_1"/>
         <child link="depth_camera_link"/>
-        <origin xyz="0.305 0 0.08" rpy="0 0 0"/>
+        <origin xyz="0.05 0 0.075" rpy="0 -1.57 0"/>
     </joint>
     <link name="depth_camera_link">
@@ -70,5 +63,5 @@
         <material>orange</material>
         <sensor name="depth_camera" type="depth">
-            <pose> 0 0 0 0 0 0 </pose>
+            <pose> 0 0 0 0 1.57 0 </pose>
             <visualize>true</visualize>
             <update_rate>10</update_rate>

File: urdf2/final_description/urdf/example_gazebo.xacro (robot description, xacro)
@@ -2,8 +2,11 @@
 <robot xmlns:xacro="http://www.ros.org/wiki/xacro">
     <gazebo>
+        <odometry_frame>odom</odometry_frame>
+        <robot_base_frame>base_link</robot_base_frame>
+        <publish_odom>true</publish_odom>
+        <publish_odom_tf>true</publish_odom_tf>
         <plugin name="ignition::gazebo::systems::JointStatePublisher"
             filename="ignition-gazebo-joint-state-publisher-system">
             <update_rate>20</update_rate>
-            <joint_name>world_to_base</joint_name>
             <joint_name>Slider_2</joint_name>
             <joint_name>Slider_6</joint_name>

File: urdf2/final_description/urdf/example_include.xacro (robot description, xacro)
@@ -1,4 +1,7 @@
 <?xml version="1.0"?>
 <robot xmlns:xacro="http://www.ros.org/wiki/xacro" >
+    <material name="black">
+        <color rgba="0 0 0 1"/>
+    </material>
     <material name="white">
         <color rgba="1 1 1 1"/>

File: urdf2/final_description/urdf/final.urdf.xacro (robot description, xacro)
@@ -7,10 +7,4 @@
 <xacro:include filename="example_gazebo.xacro" />
 <xacro:include filename="camera.xacro" />
-<link name="world"/>
-<joint name="world_to_base" type="fixed">
-  <origin xyz="0 0 0"/>
-  <parent link="world"/>
-  <child link="base_link"/>
-</joint>
 <link name="base_link">
   <inertial>
@@ -228,12 +222,20 @@
         </joint>
 </ros2_control>
+  <gazebo reference = "runner_plate_v1_1">
+    <plugin
+      filename="ignition-gazebo-imu-system"
+      name="ignition::gazebo::systems::Imu">
+    </plugin>
+    <sensor name="imu_sensor" type="imu">
+      <always_on>1</always_on>
+      <update_rate>1</update_rate>
+      <visualize>true</visualize>
+      <topic>imu</topic>
+    </sensor>
+  </gazebo>
   <gazebo>
     <plugin filename="ign_ros2_control-system" name="ign_ros2_control::IgnitionROS2ControlPlugin">
       <parameters>$(find movement)/config/ros2_controllers.yaml</parameters>
     </plugin>
-    <plugin
-      filename="ignition-gazebo-imu-system"
-      name="ignition::gazebo::systems::Imu">
-    </plugin>
   </gazebo>
 </robot>
